File: hardware/kicad/robot_canettes/MOTOR_DRIVE.kicad_sch (KiCad schematic)
At the start: 0 parts

Commit message: motor drive
Parts:
- added C1: 10uF, Capacitor_SMD:C_0805_2012Metric, symbol Device:C_Small
- added C2: 10nF, Capacitor_SMD:C_0402_1005Metric, symbol Device:C_Small
- added C3: 2.2uF, Capacitor_SMD:C_0402_1005Metric, symbol Device:C_Small
- added U2: DRV8833PWP, Package_SO:HTSSOP-16-1EP_4.4x5mm_P0.65mm_EP3.4x5mm_Mask2.46x2.31mm, symbol Driver_Motor:DRV8833PWP
Connections:
- new net: C2.2, U2.11 (VCP)
- new net: C3.2, U2.14 (VINT)
- new net GND: C1.2, C3.1, U2.13 (GND), U2.17 (GND), U2.3 (AISEN), U2.6 (BISEN)
- new net MOTOR_A_IN1: U2.16 (AIN1)
- new net MOTOR_A_IN2: U2.15 (AIN2)
- new net MOTOR_B_IN1: U2.9 (BIN1)
- new net MOTOR_B_IN2: U2.10 (BIN2)
- new net MOTOR_FAULT: U2.8 (~{FAULT})
- new net MOTOR_SLEEP: U2.1 (~{SLEEP})
- new net VM: C1.1, C2.1, U2.12 (VM)

Commit message: Update motor drive
Parts:
- removed C1: 10uF, Capacitor_SMD:C_0805_2012Metric, symbol Device:C_Small
- removed C2: 10nF, Capacitor_SMD:C_0402_1005Metric, symbol Device:C_Small
- removed C3: 2.2uF, Capacitor_SMD:C_0402_1005Metric, symbol Device:C_Small
- removed U2: DRV8833PWP, Package_SO:HTSSOP-16-1EP_4.4x5mm_P0.65mm_EP3.4x5mm_Mask2.46x2.31mm, symbol Driver_Motor:DRV8833PWP
- added C16: 10nF, Capacitor_SMD:C_0402_1005Metric, symbol Device:C_Small
- added C17: 2.2uF, Capacitor_SMD:C_0402_1005Metric, symbol Device:C_Small
- added C18: 10uF, Capacitor_SMD:C_0805_2012Metric, symbol Device:C_Small
- added C19: 100uF, Capacitor_SMD:CP_Elec_6.3x7.7, symbol Device:C_Polarized_Small
- added C20: 100uF, Capacitor_SMD:CP_Elec_6.3x5.4, symbol Device:C_Polarized_Small
- added C21, C22: 100nF, Capacitor_SMD:C_0402_1005Metric, symbol Device:C_Small
- added J6: Conn_01x03, Connector_PinHeader_2.54mm:PinHeader_1x03_P2.54mm_Vertical, symbol Connector_Generic:Conn_01x03
- added J7, J8: Conn_01x06, Connector_JST:JST_XH_S6B-XH-A-1_1x06_P2.50mm_Horizontal, symbol Connector_Generic:Conn_01x06
- added R3: 10K, Resistor_SMD:R_0402_1005Metric, symbol Device:R
- added U3: DRV8833PWP, Package_SO:HTSSOP-16-1EP_4.4x5mm_P0.65mm_EP3.4x5mm_Mask2.46x2.31mm, symbol Driver_Motor:DRV8833PWP
Connections:
- net GND: now also C17.1, C18.2, C19.2, C20.2, C21.2, C22.2, J6.1 (Pin_1), J7.2 (Pin_2), J8.2 (Pin_2), U3.13 (GND), U3.17 (GND), U3.3 (AISEN), U3.6 (BISEN)
- net MOTOR_A_IN1: now also U3.16 (AIN1)
- net MOTOR_A_IN2: now also U3.15 (AIN2)
- net MOTOR_B_IN1: now also U3.9 (BIN1)
- net MOTOR_B_IN2: now also U3.10 (BIN2)
- net MOTOR_FAULT: now also R3.2, U3.8 (~{FAULT})
- net MOTOR_SLEEP: now also U3.1 (~{SLEEP})
- net VM: now also C16.1, C18.1, C19.1, C21.1, U3.12 (VM)
- new net: C16.2, U3.11 (VCP)
- new net: J8.1 (Pin_1), U3.2 (AOUT1)
- new net: J8.6 (Pin_6), U3.4 (AOUT2)
- new net: C17.2, U3.14 (VINT)
- new net: J7.6 (Pin_6), U3.5 (BOUT2)
- new net: J7.1 (Pin_1), U3.7 (BOUT1)
- new net +3.3V: R3.1
- new net +3V3: J7.5 (Pin_5), J8.5 (Pin_5)
- new net 5V: C20.1, C22.1, J6.2 (Pin_2)
- new net MOTOR_A_C1: J8.3 (Pin_3)
- new net MOTOR_A_C2: J8.4 (Pin_4)
- new net MOTOR_B_C1: J7.3 (Pin_3)
- new net MOTOR_B_C2: J7.4 (Pin_4)
- new net SERVO1_PWM: J6.3 (Pin_3)
Other:
- note added: "Bloc DRV8833"
- note added: "Bloc servo"
- note added: "SERVO POWER DECOUPLING"

Commit message: MAJ schema MCU/sensors
Parts:
- removed C16: 10nF, Capacitor_SMD:C_0402_1005Metric, symbol Device:C_Small
- removed C17: 2.2uF, Capacitor_SMD:C_0402_1005Metric, symbol Device:C_Small
- removed C19: 100uF, Capacitor_SMD:CP_Elec_6.3x7.7, symbol Device:C_Polarized_Small
- removed C20: 100uF, Capacitor_SMD:CP_Elec_6.3x5.4, symbol Device:C_Polarized_Small
- removed C21, C22: 100nF, Capacitor_SMD:C_0402_1005Metric, symbol Device:C_Small
- added C19: 2.2uF, Capacitor_SMD:C_0402_1005Metric, symbol Device:C_Small
- added C20: 10uF, Capacitor_SMD:C_0805_2012Metric, symbol Device:C_Small
- added C21: 100uF, Capacitor_SMD:CP_Elec_6.3x7.7, symbol Device:C_Polarized_Small
- added C22: 100uF, Capacitor_SMD:CP_Elec_6.3x5.4, symbol Device:C_Polarized_Small
- added C23, C24: 100nF, Capacitor_SMD:C_0402_1005Metric, symbol Device:C_Small
- C18: value 10uF -> 10nF; footprint Capacitor_SMD:C_0805_2012Metric -> Capacitor_SMD:C_0402_1005Metric; JLCPCB Part # C380332 -> C15195
Connections:
- net 5V: now also C22.1, C24.1
- net GND: now also C19.1, C20.2, C21.2, C22.2, C23.2, C24.2; no longer C18.2
- net VM: now also C20.1, C21.1, C23.1
- net at U3.11 (VCP): now also C18.2
- net at U3.14 (VINT): now also C19.2

Commit message: MAJ connecteur TOF2 (J10) et resistances pull-up
Connections:
- net 5V renamed +5V
Changed lines of the file:
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@@
-	)
-	(junction
-		(at 106.68 62.23)
-		(diameter 0)
-		(color 0 0 0 0)
 	)
 	(junction
@@
 	(wire
 		(pts
-			(xy 106.68 62.23) (xy 107.95 62.23)
+			(xy 105.41 62.23) (xy 107.95 62.23)
 		)
 		(stroke
@@
 		(pts
 			(xy 120.65 80.01) (xy 120.65 82.55)
-		)
-		(stroke
-			(width 0)
-			(type default)
-		)
-	)
-	(wire
-		(pts
-			(xy 105.41 62.23) (xy 106.68 62.23)
 		)
 		(stroke
@@
 			)
 			(justify left bottom)
-		)
-	)
-	(hierarchical_label "5V"
-		(shape input)
-		(at 55.88 127 0)
-		(effects
-			(font
-				(size 1.27 1.27)
-			)
-			(justify left)
 		)
 	)
@@
 			)
 			(justify right)
-		)
-	)
-	(hierarchical_label "5V"
-		(shape input)
-		(at 163.83 130.81 90)
-		(effects
-			(font
-				(size 1.27 1.27)
-			)
-			(justify left)
 		)
 	)
@@
 	)
 	(symbol
+		(lib_id "power:+5V")
+		(at 55.88 127 270)
+		(unit 1)
+		(body_style 1)
+		(exclude_from_sim no)
+		(in_bom yes)
+		(on_board yes)
+		(in_pos_files yes)
+		(dnp no)
+		(fields_autoplaced yes)
+		(property "Reference" "#PWR073"
+			(at 52.07 127 0)
+			(hide yes)
+			(show_name no)
+			(do_not_autoplace no)
+			(effects
+				(font
+					(size 1.27 1.27)
+				)
+			)
+		)
+		(property "Value" "+5V"
+			(at 59.69 126.9999 90)
+			(show_name no)
+			(do_not_autoplace no)
+			(effects
+				(font
+					(size 1.27 1.27)
+				)
+				(justify left)
+			)
+		)
+		(property "Footprint" ""
+			(at 55.88 127 0)
+			(hide yes)
+			(show_name no)
+			(do_not_autoplace no)
+			(effects
+				(font
+					(size 1.27 1.27)
+				)
+			)
+		)
+		(property "Datasheet" ""
+			(at 55.88 127 0)
+			(hide yes)
+			(show_name no)
+			(do_not_autoplace no)
+			(effects
+				(font
+					(size 1.27 1.27)
+				)
+			)
+		)
+		(property "Description" "Power symbol creates a global label with name \"+5V\""
+			(at 55.88 127 0)
+			(hide yes)
+			(show_name no)
+			(do_not_autoplace no)
+			(effects
+				(font
+					(size 1.27 1.27)
+				)
+			)
+		)
+		(pin "1"
+		)
+		(instances
+			(project "robot_canettes"
+				(path "/67ea9330-6bd8-4bfd-bb5f-e77247705b59/7ba74d93-6812-4e1d-b9dd-cd37ba11b0d3"
+					(reference "#PWR073")
+					(unit 1)
+				)
+			)
+		)
+	)
+	(symbol
 		(lib_id "power:GND")
 		(at 120.65 82.55 0)
@@
 				(path "/67ea9330-6bd8-4bfd-bb5f-e77247705b59/7ba74d93-6812-4e1d-b9dd-cd37ba11b0d3"
 					(reference "R3")
-					(unit 1)
-				)
-			)
-		)
-	)
-	(symbol
-		(lib_id "power:PWR_FLAG")
-		(at 106.68 62.23 0)
-		(unit 1)
-		(body_style 1)
-		(exclude_from_sim no)
-		(in_bom yes)
-		(on_board yes)
-		(in_pos_files yes)
-		(dnp no)
-		(fields_autoplaced yes)
-		(property "Reference" "#FLG06"
-			(at 106.68 60.325 0)
-			(hide yes)
-			(show_name no)
-			(do_not_autoplace no)
-			(effects
-				(font
-					(size 1.27 1.27)
-				)
-			)
-		)
-		(property "Value" "PWR_FLAG"
-			(at 106.68 57.15 0)
-			(show_name no)
-			(do_not_autoplace no)
-			(effects
-				(font
-					(size 1.27 1.27)
-				)
-			)
-		)
-		(property "Footprint" ""
-			(at 106.68 62.23 0)
-			(hide yes)
-			(show_name no)
-			(do_not_autoplace no)
-			(effects
-				(font
-					(size 1.27 1.27)
-				)
-			)
-		)
-		(property "Datasheet" ""
-			(at 106.68 62.23 0)
-			(hide yes)
-			(show_name no)
-			(do_not_autoplace no)
-			(effects
-				(font
-					(size 1.27 1.27)
-				)
-			)
-		)
-		(property "Description" "Special symbol for telling ERC where power comes from"
-			(at 106.68 62.23 0)
-			(hide yes)
-			(show_name no)
-			(do_not_autoplace no)
-			(effects
-				(font
-					(size 1.27 1.27)
-				)
-			)
-		)
-		(pin "1"
-		)
-		(instances
-			(project "robot_canettes"
-				(path "/67ea9330-6bd8-4bfd-bb5f-e77247705b59/7ba74d93-6812-4e1d-b9dd-cd37ba11b0d3"
-					(reference "#FLG06")
 					(unit 1)
 				)
@@
 					(unit 1)
 				)
+			)
+		)
+	)
+	(symbol
+		(lib_id "power:+5V")
+		(at 163.83 130.81 0)
+		(unit 1)
+		(body_style 1)
+		(exclude_from_sim no)
+		(in_bom yes)
+		(on_board yes)
+		(in_pos_files yes)
+		(dnp no)
+		(fields_autoplaced yes)
+		(property "Reference" "#PWR072"
+			(at 163.83 134.62 0)
+			(hide yes)
+			(show_name no)
+			(do_not_autoplace no)
+			(effects
+				(font
+					(size 1.27 1.27)
+				)
+			)
+		)
+		(property "Value" "+5V"
+			(at 163.83 125.73 0)
+			(show_name no)
+			(do_not_autoplace no)
+			(effects
+				(font
+					(size 1.27 1.27)
+				)
+			)
+		)
+		(property "Footprint" ""
+			(at 163.83 130.81 0)
+			(hide yes)
+			(show_name no)
+			(do_not_autoplace no)
+			(effects
+				(font
+					(size 1.27 1.27)
+				)
+			)
+		)
+		(property "Datasheet" ""
+			(at 163.83 130.81 0)
+			(hide yes)
+			(show_name no)
+			(do_not_autoplace no)
+			(effects
+				(font
+					(size 1.27 1.27)
+				)
+			)
+		)
+		(property "Description" "Power symbol creates a global label with name \"+5V\""
+			(at 163.83 130.81 0)
+			(hide yes)
+			(show_name no)
+			(do_not_autoplace no)
+			(effects
+				(font
+					(size 1.27 1.27)
+				)
+			)
+		)
+		(pin "1"
+		)
+		(instances
+			(project "robot_canettes"
+				(path "/67ea9330-6bd8-4bfd-bb5f-e77247705b59/7ba74d93-6812-4e1d-b9dd-cd37ba11b0d3"
+					(reference "#PWR072")
+					(unit 1)
+				)
