File: hardware/kicad/robot_canettes/MOTOR_DRIVE.kicad_sch (KiCad schematic)
At the start: 12 parts, among them J6 Conn_01x03, J7 Conn_01x06, J8 Conn_01x06, U3 DRV8833PWP

Commit message: MOTOR_DRIVE
Parts:
- removed C16: 10nF, Capacitor_SMD:C_0402_1005Metric, symbol Device:C_Small
- removed C17: 2.2uF, Capacitor_SMD:C_0402_1005Metric, symbol Device:C_Small
- removed C19: 100uF, Capacitor_SMD:CP_Elec_6.3x7.7, symbol Device:C_Polarized_Small
- removed C20: 100uF, Capacitor_SMD:CP_Elec_6.3x5.4, symbol Device:C_Polarized_Small
- removed C21, C22: 100nF, Capacitor_SMD:C_0402_1005Metric, symbol Device:C_Small
- added C19: 2.2uF, Capacitor_SMD:C_0402_1005Metric, symbol Device:C_Small
- added C20: 10uF, Capacitor_SMD:C_0805_2012Metric, symbol Device:C_Small
- added C21: 100uF, Capacitor_SMD:CP_Elec_6.3x7.7, symbol Device:C_Polarized_Small
- added C22: 100uF, Capacitor_SMD:CP_Elec_6.3x5.4, symbol Device:C_Polarized_Small
- added C23, C24, C35, C37: 100nF, Capacitor_SMD:C_0402_1005Metric, symbol Device:C_Small
- added R13, R21: 200m, Resistor_SMD:R_2512_6332Metric, symbol Device:R
- C18: value 10uF -> 10nF; footprint Capacitor_SMD:C_0805_2012Metric -> Capacitor_SMD:C_0402_1005Metric; JLCPCB Part # C380332 -> C15195
Connections:
- net +3V3 is gone; now on net GND: J7.5 (Pin_5), J8.5 (Pin_5)
- net +3.3V: now also J7.2 (Pin_2), J8.2 (Pin_2), C35.1, C37.1
- net GND: now also C19.1, C20.2, C21.2, C22.2, C23.2, C24.2, C35.2, C37.2, R13.1, R21.1; no longer C18.2, J7.2 (Pin_2), J8.2 (Pin_2), U3.3 (AISEN), U3.6 (BISEN)
- net VM: now also C20.1, C21.1, C23.1
- net at U3.11 (VCP): now also C18.2
- net at U3.14 (VINT): now also C19.2
- net 5V renamed +5V
- net +5V: now also C22.1, C24.1
- new net: R13.2, U3.3 (AISEN)
- new net: R21.2, U3.6 (BISEN)
