File: hardware/kicad/robot_canettes/MOTOR_DRIVE.kicad_sch (KiCad schematic)
At the start: 14 parts, among them J6 Conn_01x03, J7 Conn_01x06, J8 Conn_01x06, U3 DRV8833PWP

Commit message: Mise à jour de l'emplacement des composants
Parts:
- J7, J8: footprint Connector_JST:JST_XH_S6B-XH-A-1_1x06_P2.50mm_Horizontal -> Connector_JST:JST_PH_B6B-PH-K_1x06_P2.00mm_Vertical
Connections:
- net GND: now reaches J6.1 (Pin_1)
- net GND: now also C19.1, C20.2, C24.2, C34.2, J8.2 (Pin_2), R17.2, R18.2, U3.13 (GND), U3.17 (GND)
Changed lines of the file:
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@@
 			)
 		)
-		(property "Value" ""
+		(property "Value" "GND"
 			(at 111.76 50.8 0)
+			(hide yes)
 			(show_name no)
 			(do_not_autoplace no)
@@
 			)
 		)
-		(property "Value" ""
+		(property "Value" "GND"
 			(at 120.65 86.614 0)
+			(hide yes)
 			(show_name no)
 			(do_not_autoplace no)
@@
 			)
 		)
-		(property "Value" ""
+		(property "Value" "GND"
 			(at 143.51 59.69 0)
+			(hide yes)
 			(show_name no)
 			(do_not_autoplace no)
@@
 			)
 		)
-		(property "Value" ""
+		(property "Value" "GND"
 			(at 188.214 71.374 0)
+			(hide yes)
 			(show_name no)
 			(do_not_autoplace no)
@@
 			)
 		)
-		(property "Value" ""
+		(property "Value" "GND"
 			(at 181.61 142.24 0)
+			(hide yes)
 			(show_name no)
 			(do_not_autoplace no)
@@
 			)
 		)
-		(property "Value" ""
+		(property "Value" "GND"
 			(at 91.44 144.78 0)
+			(hide yes)
 			(show_name no)
 			(do_not_autoplace no)
@@
 			)
 		)
-		(property "Footprint" "Connector_JST:JST_XH_S6B-XH-A-1_1x06_P2.50mm_Horizontal"
+		(property "Footprint" "Connector_JST:JST_PH_B6B-PH-K_1x06_P2.00mm_Vertical"
 			(at 228.6 72.39 0)
 			(hide yes)
@@
 			)
 		)
-		(property "Footprint" "Connector_JST:JST_XH_S6B-XH-A-1_1x06_P2.50mm_Horizontal"
+		(property "Footprint" "Connector_JST:JST_PH_B6B-PH-K_1x06_P2.00mm_Vertical"
 			(at 170.18 77.47 0)
 			(hide yes)
@@
 			)
 		)
-		(property "Value" ""
+		(property "Value" "GND"
 			(at 49.53 74.93 0)
-			(show_name no)
-			(do_not_autoplace no)
+			(hide yes)
+			(show_name no)
+			(do_not_autoplace no)

Commit message: Final PCB LAYOUT
Parts:
- J6: JLCPCB Part # C49257 -> C131339
- J7, J8: JLCPCB Part # C265069 -> C131342
Changed lines of the file:
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@@
 			)
 		)
-		(property "JLCPCB Part #" "C49257"
+		(property "JLCPCB Part #" "C131339"
 			(at 170.18 134.62 0)
 			(hide yes)
@@
 			)
 		)
-		(property "JLCPCB Part #" "C265069"
+		(property "JLCPCB Part #" "C131342"
 			(at 228.6 72.39 0)
 			(hide yes)
@@
 			)
 		)
-		(property "JLCPCB Part #" "C265069"
+		(property "JLCPCB Part #" "C131342"
 			(at 170.18 77.47 0)
 			(hide yes)

Commit message: Mise a jour des schemas, layout final, routage et génération des fichiers de fabrication de la carte
Parts:
- C24: JLCPCB Part # C1525 -> C1525
- C34: JLCPCB Part # (none) -> C52923
- R17, R18: JLCPCB PART # C1727756 -> (none); JLCPCB Part # (none) -> C5127778
- R3: JLCPCB Part # C844714 -> C25744
- renumbered J7 to M1, J8 to M2, J6 to Servo1
Changed lines of the file:
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@@
 		(dnp no)
 		(property "Reference" "C18"
-			(at 94.234 55.372 90)
+			(at 97.536 54.356 90)
 			(show_name no)
 			(do_not_autoplace no)
@@
 		)
 		(property "Value" "10n"
-			(at 97.79 54.102 90)
+			(at 100.838 58.674 90)
 			(show_name no)
 			(do_not_autoplace no)
@@
 		(dnp no)
 		(fields_autoplaced yes)
-		(property "Reference" "J6"
+		(property "Reference" "Servo1"
 			(at 170.18 125.73 0)
 			(show_name no)
@@
 			(project "robot_canettes"
 				(path "/67ea9330-6bd8-4bfd-bb5f-e77247705b59/7ba74d93-6812-4e1d-b9dd-cd37ba11b0d3"
-					(reference "J6")
+					(reference "Servo1")
 					(unit 1)
 				)
@@
 			)
 		)
-		(property "JLCPCB Part #" "C844714"
+		(property "JLCPCB Part #" "C25744"
 			(at 180.848 52.324 0)
 			(hide yes)
@@
 			)
 		)
-		(property "JLCPCB Part #" "C1525 "
+		(property "JLCPCB Part #" "C1525"
 			(at 99.06 135.89 0)
 			(hide yes)
@@
 			)
 		)
+		(property "JLCPCB Part #" "C52923"
+			(at 82.55 135.89 0)
+			(hide yes)
+			(show_name no)
+			(do_not_autoplace no)
+			(effects
+				(font
+					(size 1.27 1.27)
+				)
+			)
+		)
 		(pin "1"
 		)
@@
 		(dnp no)
 		(fields_autoplaced yes)
-		(property "Reference" "J8"
+		(property "Reference" "M2"
 			(at 231.14 72.3899 0)
 			(show_name no)
@@
 			(project "robot_canettes"
 				(path "/67ea9330-6bd8-4bfd-bb5f-e77247705b59/7ba74d93-6812-4e1d-b9dd-cd37ba11b0d3"
-					(reference "J8")
+					(reference "M2")
 					(unit 1)
 				)
@@
 		(in_pos_files yes)
 		(dnp no)
-		(property "Reference" "J7"
+		(property "Reference" "M1"
 			(at 172.212 82.042 0)
 			(show_name no)
@@
 			(project "robot_canettes"
 				(path "/67ea9330-6bd8-4bfd-bb5f-e77247705b59/7ba74d93-6812-4e1d-b9dd-cd37ba11b0d3"
-					(reference "J7")
+					(reference "M1")
 					(unit 1)
 				)
@@
 			)
 		)
-		(property "JLCPCB PART #" "C1727756"
+		(property "JLCPCB Part #" "C5127778"
 			(at 49.53 66.04 0)
 			(hide yes)
@@
 			)
 		)
-		(property "JLCPCB PART #" "C1727756"
+		(property "JLCPCB Part #" "C5127778"
 			(at 59.69 66.04 0)
 			(hide yes)
