File: hardware/kicad/robot_canettes/POWER_MANAGEMENT.kicad_sch (KiCad schematic)
At the start: 0 parts

Commit message: Mise à jour de la feuille POWER Management
Parts:
- added C25, C26, C27: 1u, Capacitor_SMD:C_0402_1005Metric, symbol Device:C_Small
- added C28: 47n, Capacitor_SMD:C_0402_1005Metric, symbol Device:C_Small
- added C29: 4u7, Capacitor_SMD:C_0402_1005Metric, symbol Device:C_Small
- added C30, C31, C32, C33: 10u, Capacitor_SMD:C_0402_1005Metric, symbol Device:C_Small
- added C34: 0u47, Capacitor_SMD:C_0402_1005Metric, symbol Device:C_Small
- added D1: STATUS, LED_SMD:LED_0603_1608Metric, symbol Device:LED_Small
- added J4: USB_C_Receptacle_USB2.0_16P, Connector_USB:USB_C_Receptacle_GCT_USB4105-xx-A_16P_TopMnt_Horizontal, symbol Connector:USB_C_Receptacle_USB2.0_16P
- added J5: Conn_01x02_Pin, Connector_JST:JST_PH_B2B-PH-K_1x02_P2.00mm_Vertical, symbol Connector:Conn_01x02_Pin
- added L1: 2u2, Inductor_SMD:L_2010_5025Metric_Pad1.52x2.65mm_HandSolder, symbol Device:L_Small
- added Q1: 2N7002, Package_TO_SOT_SMD:SOT-23, symbol Transistor_FET:2N7002
- added R10, R11, R15, R16, R6, R7, R8: 10K, Resistor_SMD:R_0402_1005Metric, symbol Device:R_Small
- added R12: 260, Resistor_SMD:R_0402_1005Metric, symbol Device:R_Small
- added R13: 100K, Resistor_SMD:R_0402_1005Metric, symbol Device:R_Small
- added R14: 2K2, Resistor_SMD:R_0402_1005Metric, symbol Device:R_Small
- added R17, R18, R20, R4, R5: 5K1, Resistor_SMD:R_0402_1005Metric, symbol Device:R_Small
- added R19: 100, Resistor_SMD:R_1206_3216Metric, symbol Device:R
- added R9: 100, Resistor_SMD:R_0402_1005Metric, symbol Device:R_Small
- added SW1, SW2: (no value), Button_Switch_SMD:SW_SPST_Omron_B3FS-101xP, symbol Switch:SW_Omron_B3FS
- added U4: AP2112K-3.3, Package_TO_SOT_SMD:SOT-23-5, symbol Regulator_Linear:AP2112K-3.3
- added U5: USBLC6-2SC6, Package_TO_SOT_SMD:SOT-23-6, symbol Power_Protection:USBLC6-2SC6
- added U6: BQ25895RTW, Package_DFN_QFN:Texas_RTW_WQFN-24-1EP_4x4mm_P0.5mm_EP2.7x2.7mm_ThermalVias, symbol Battery_Management:BQ25895RTW
- added U7: BQ27441-G1, Package_SON:Texas_S-PDSO-N12, symbol Battery_Management:BQ27441-G1
Connections:
- new net: C34.1, U7.5 (V_{DD})
- new net: U7.13 (PAD), U7.3 (V_{SS})
- new net: J4.B5 (CC2), R4.1
- new net: R13.1, SW2.2, U4.3 (EN)
- new net: J4.A5 (CC1), R5.1
- new net: R15.1, R16.1, U6.11 (TS)
- new net: C29.1, R15.2, U6.22 (REGN)
- new net: SW1.2, U6.12 (~{QON})
- new net: D1.1 (K), R14.1
- new net: R14.2, U6.4 (STAT)
- new net: R12.1, U6.10 (ILIM)
- new net: U6.17 (PGND), U6.18 (PGND), U6.25 (PGND)
- new net: C28.1, L1.1, U6.19 (SW), U6.20 (SW)
- new net: C28.2, U6.21 (BTST)
- new net: Q1.3 (D), R8.2, U6.8 (OTG)
- new net: Q1.1 (G), R10.1, R9.2
- new net: Q1.2 (S), R10.2
- new net +BATT: J5.2 (Pin_2), R19.1, U7.6 (BAT), U7.8 (SRP)
- new net 3V3: C26.1, R11.1, R17.1, R18.1, R20.1, R6.1, R7.1, U4.5 (VOUT)
- new net 5V: C30.2, U6.23 (PMID)
- new net Charger_D+: U5.4 (I/O2), U6.2 (D+)
- new net Charger_D-: U5.6 (I/O1)
- new net Chargeur_D-: U6.3 (D-)
- new net GAUGE_INT: R20.2, U7.12 (GPOUT)
- new net GND: C29.2, J4.A1 (GND), J4.A12 (GND), J4.B1 (GND), J4.B12 (GND), J4.SH (SHIELD), R12.2, R4.2, R5.2, U5.2 (GND)
- new net I2C3_SCL: R17.2, R6.2, U6.6 (SDA), U7.2 (SCL)
- new net I2C3_SDA: R11.2, R18.2, U6.5 (SCL), U7.1 (SDA)
- new net INT: R7.2, U6.7 (~{INT})
- new net SRN: C32.1, R19.2, U6.13 (BAT), U6.14 (BAT), U7.7 (SRN)
- new net SYS: C25.1, C31.1, C33.1, D1.2 (A), L1.2, R8.1, SW2.1, U4.1 (VIN), U6.15 (SYS), U6.16 (SYS)
- new net USB_D+: J4.A6 (D+), J4.B6 (D+), U5.3 (I/O2)
- new net USB_D-: J4.A7 (D-), J4.B7 (D-), U5.1 (I/O1)
- new net VBUS: C27.1, J4.A4 (VBUS), J4.A9 (VBUS), J4.B4 (VBUS), J4.B9 (VBUS), R9.1, U5.5 (VBUS), U6.1 (VBUS)
- no-connect marks 0 -> 3
Other:
- note added: "3V3 Power"
- note added: "Battery charger"
- note added: "Connecteur USB, charge de la pile"
- note added: "ESD Protection"
- note added: "Fuel Gauge"

Commit message: MAJ connecteur TOF2 (J10) et resistances pull-up
Parts:
- removed R13: 100K, Resistor_SMD:R_0402_1005Metric, symbol Device:R_Small
- removed SW2: (no value), Button_Switch_SMD:SW_SPST_Omron_B3FS-101xP, symbol Switch:SW_Omron_B3FS
Connections:
- net Charger_D- is gone; now on net Chargeur_D-: U5.6 (I/O1)
- net +BATT: no longer R19.1
- net SRN: no longer R19.2
- net SYS: now also U4.3 (EN)
- net 3V3 renamed +3.3V
- net 5V renamed +5V
Other:
- moved on the sheet: C25, C26, C27, C28, C29, C30, C31, C32, C33, C34, D1, J5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
