File: hardware/kicad/robot_canettes/POWER_MANAGEMENT.kicad_sch (KiCad schematic)
At the start: 54 parts, among them J4 USB_C_Receptacle_USB2.0_16P, J5 Conn_01x02_Pin, Q1 2N7002, Q2 Q_PMOS, Q5 Q_PNP_CurrentMirror, U4 AP2112K-3.3, U5 bq27220, U9 BQ25896RTWR

Commit message: Mise à jour de l'emplacement des composants
Connections:
- net GND: now also C25.2, C26.2, C27.2, C30.1, C31.2, C32.2, C33.2, C42.1, J5.1 (Pin_1), Q1.2 (S), R10.2, R16.2, R22.2, R24.2, R25.2, R27.2, SW1.1, U4.2 (GND), U5.B2 (VSS), U9.17 (PGND), U9.18 (PGND), U9.25 (PGND), U9.9 (~{CE})
Changed lines of the file:
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@@
 			)
 		)
-		(property "Value" ""
+		(property "Value" "GND"
 			(at 78.74 137.16 0)
+			(hide yes)
 			(show_name no)
 			(do_not_autoplace no)
@@
 			)
 		)
-		(property "Value" ""
+		(property "Value" "GND"
 			(at 172.72 129.54 0)
+			(hide yes)
 			(show_name no)
 			(do_not_autoplace no)
@@
 			)
 		)
-		(property "Value" ""
+		(property "Value" "GND"
 			(at 97.79 180.34 0)
+			(hide yes)
 			(show_name no)
 			(do_not_autoplace no)
@@
 			)
 		)
-		(property "Value" ""
+		(property "Value" "GND"
 			(at 214.63 59.69 0)
+			(hide yes)
 			(show_name no)
 			(do_not_autoplace no)
@@
 			)
 		)
-		(property "Value" ""
+		(property "Value" "GND"
 			(at 83.82 163.83 0)
+			(hide yes)
 			(show_name no)
 			(do_not_autoplace no)
@@
 			)
 		)
-		(property "Value" ""
+		(property "Value" "GND"
 			(at 157.48 67.31 0)
+			(hide yes)
 			(show_name no)
 			(do_not_autoplace no)
@@
 			)
 		)
-		(property "Value" ""
+		(property "Value" "GND"
 			(at 139.7 160.02 0)
+			(hide yes)
 			(show_name no)
 			(do_not_autoplace no)
@@
 			)
 		)
-		(property "Value" ""
+		(property "Value" "GND"
 			(at 168.91 185.42 0)
+			(hide yes)
 			(show_name no)
 			(do_not_autoplace no)
@@
 			)
 		)
-		(property "Value" ""
+		(property "Value" "GND"
 			(at 128.27 69.85 0)
+			(hide yes)
 			(show_name no)
 			(do_not_autoplace no)
@@
 			)
 		)
-		(property "Value" ""
+		(property "Value" "GND"
 			(at 73.66 181.61 0)
+			(hide yes)
 			(show_name no)
 			(do_not_autoplace no)
@@
 			)
 		)
-		(property "Value" ""
+		(property "Value" "GND"
 			(at 139.7 69.85 0)
+			(hide yes)
 			(show_name no)
 			(do_not_autoplace no)
@@
 			)
 		)
-		(property "Value" ""
+		(property "Value" "GND"
 			(at 132.08 186.69 0)
+			(hide yes)
 			(show_name no)
 			(do_not_autoplace no)
@@
 		(in_pos_files yes)
 		(dnp no)
-		(fields_autoplaced yes)
 		(property "Reference" "#PWR058"
 			(at 133.35 147.32 0)
@@
 			)
 		)
-		(property "Value" ""
-			(at 133.35 146.05 0)
+		(property "Value" "GND"
+			(at 133.35 144.526 0)
+			(hide yes)
 			(show_name no)
 			(do_not_autoplace no)
@@
 		(in_pos_files yes)
 		(dnp no)
-		(fields_autoplaced yes)
 		(property "Reference" "#PWR059"
 			(at 129.54 161.29 0)
@@
 			)
 		)
-		(property "Value" ""
+		(property "Value" "GND"
 			(at 129.54 160.02 0)
+			(hide yes)
 			(show_name no)
 			(do_not_autoplace no)
@@
 			)
 		)
-		(property "Value" ""
+		(property "Value" "GND"
 			(at 254 76.2 0)
+			(hide yes)
 			(show_name no)
 			(do_not_autoplace no)
@@
 			)
 		)
-		(property "Value" ""
+		(property "Value" "GND"
 			(at 111.76 186.69 0)
+			(hide yes)
 			(show_name no)
 			(do_not_autoplace no)
@@
 			)
 		)
-		(property "Value" ""
+		(property "Value" "GND"
 			(at 232.41 166.37 0)
+			(hide yes)
 			(show_name no)
 			(do_not_autoplace no)
@@
 			)
 		)
-		(property "Value" ""
+		(property "Value" "GND"
 			(at 254 166.37 0)
+			(hide yes)
 			(show_name no)
 			(do_not_autoplace no)
@@
 			)
 		)
-		(property "Value" ""
+		(property "Value" "GND"
 			(at 90.17 69.85 0)
+			(hide yes)
 			(show_name no)
 			(do_not_autoplace no)
@@
 			)
 		)
-		(property "Value" ""
+		(property "Value" "GND"
 			(at 53.34 195.58 0)
+			(hide yes)
 			(show_name no)
 			(do_not_autoplace no)

Commit message: Final PCB LAYOUT
Parts:
- J5: JLCPCB Part # (none) -> C131337
- R26: JLCPCB Part # C500740 -> C2903499
Changed lines of the file:
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@@
 			)
 		)
-		(property "JLCPCB Part #" "C500740"
+		(property "JLCPCB Part #" "C2903499"
 			(at 152.4 158.75 90)
 			(hide yes)
@@
 			(at 176.53 161.29 0)
 			(hide yes)
+			(show_name no)
+			(do_not_autoplace no)
+			(effects
+				(font
+					(size 1.27 1.27)
+				)
+			)
+		)
+		(property "JLCPCB Part #" "C131337"
+			(at 176.53 161.29 0)
+			(hide yes)

Commit message: Mise a jour des schemas, layout final, routage et génération des fichiers de fabrication de la carte
Parts:
- C37: JLCPCB Part # C107370 -> C12530
- D2, D3, D4: JLCPCB Part # C72043 -> C12624
- Q1: JLCPCB Part # C8485 -> C8545
- R10, R11, R15, R16, R20, R23, R6, R7, R8: JLCPCB Part # C844714 -> C25744
- renumbered J5 to Battery1, J4 to Charging1
Changed lines of the file:
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@@
 			)
 		)
-		(property "JLCPCB Part #" "C844714"
+		(property "JLCPCB Part #" "C25744"
 			(at 45.72 140.97 0)
 			(hide yes)
@@
 			)
 		)
-		(property "JLCPCB Part #" "C72043"
+		(property "JLCPCB Part #" "C12624"
 			(at 172.72 111.76 90)
 			(hide yes)
@@
 			)
 		)
-		(property "JLCPCB Part #" "C844714"
+		(property "JLCPCB Part #" "C25744"
 			(at 111.76 168.91 0)
 			(hide yes)
@@
 		(dnp no)
 		(fields_autoplaced yes)
-		(property "Reference" "J4"
+		(property "Reference" "Charging1"
 			(at 35.56 31.75 0)
 			(show_name no)
@@
 			(project "robot_canettes"
 				(path "/67ea9330-6bd8-4bfd-bb5f-e77247705b59/0d2e62ed-6bf0-41ca-b0b9-c6fd2c3353c4"
-					(reference "J4")
+					(reference "Charging1")
 					(unit 1)
 				)
@@
 			)
 		)
-		(property "JLCPCB Part #" "C107370"
+		(property "JLCPCB Part #" "C12530 "
 			(at 275.59 59.69 0)
 			(hide yes)
@@
 			)
 		)
-		(property "JLCPCB Part #" "C844714"
+		(property "JLCPCB Part #" "C25744"
 			(at 36.83 140.97 0)
 			(hide yes)
@@
 		(in_pos_files yes)
 		(dnp no)
-		(fields_autoplaced yes)
 		(property "Reference" "C42"
-			(at 212.09 52.0701 0)
+			(at 212.598 47.498 0)
 			(show_name no)
 			(do_not_autoplace no)
@@
 			)
 		)
-		(property "JLCPCB Part #" "C844714"
+		(property "JLCPCB Part #" "C25744"
 			(at 187.96 57.15 0)
 			(hide yes)
@@
 			)
 		)
-		(property "JLCPCB Part #" "C844714"
+		(property "JLCPCB Part #" "C25744"
 			(at 54.61 140.97 0)
 			(hide yes)
@@
 		(dnp no)
 		(fields_autoplaced yes)
-		(property "Reference" "J5"
+		(property "Reference" "Battery1"
 			(at 177.8 158.7499 0)
 			(show_name no)
@@
 			(project "robot_canettes"
 				(path "/67ea9330-6bd8-4bfd-bb5f-e77247705b59/0d2e62ed-6bf0-41ca-b0b9-c6fd2c3353c4"
-					(reference "J5")
+					(reference "Battery1")
 					(unit 1)
 				)
@@
 			)
 		)
-		(property "JLCPCB Part #" "C844714"
+		(property "JLCPCB Part #" "C25744"
 			(at 57.15 168.91 0)
 			(hide yes)
@@
 			)
 		)
-		(property "JLCPCB Part #" "C844714"
+		(property "JLCPCB Part #" "C25744"
 			(at 229.87 71.12 0)
 			(hide yes)
@@
 			)
 		)
-		(property "JLCPCB Part #" "C72043"
+		(property "JLCPCB Part #" "C12624"
 			(at 67.31 120.65 90)
 			(hide yes)
@@
 			)
 		)
-		(property "JLCPCB Part #" "C72043"
+		(property "JLCPCB Part #" "C12624"
 			(at 157.48 49.53 90)
 			(hide yes)
@@
 			)
 		)
-		(property "JLCPCB Part #" "C844714"
+		(property "JLCPCB Part #" "C25744"
 			(at 111.76 177.8 0)
 			(hide yes)
@@
 			)
 		)
-		(property "JLCPCB Part #" "C844714"
+		(property "JLCPCB Part #" "C25744"
 			(at 45.72 186.69 0)
 			(hide yes)
@@
 			)
 		)
-		(property "JLCPCB Part #" "C8485"
+		(property "JLCPCB Part #" "C8545"
 			(at 54.61 180.34 0)
 			(hide yes)
