File: hardware/kicad/robot_canettes/robot_canettes.kicad_sch (KiCad schematic)
At the start: 0 parts

Commit message: Creation de la hierarchie des 3 feuilles (power, mcu_sensors, motor_drive)
Other:
- added sheet MCU_AND_SENSORS (MCU_AND_SENSORS.kicad_sch)
- added sheet MOTOR_DRIVE (MOTOR_DRIVE.kicad_sch)
- added sheet POWER_MANAGEMENT (POWER_MANAGEMENT.kicad_sch)
Changed lines of the file:
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@@
 	(generator_version "10.0")
 	(paper "A4")
+	(sheet
+		(at 107.95 35.56)
+		(size 78.74 128.27)
+		(exclude_from_sim no)
+		(in_bom yes)
+		(on_board yes)
+		(dnp no)
+		(fields_autoplaced yes)
+		(stroke
+			(width 0.1524)
+			(type solid)
+		)
+		(fill
+			(color 0 0 0 0)
+		)
+		(property "Sheetname" "POWER_MANAGEMENT"
+			(at 107.95 34.8484 0)
+			(show_name no)
+			(do_not_autoplace no)
+			(effects
+				(font
+					(size 1.27 1.27)
+				)
+				(justify left bottom)
+			)
+		)
+		(property "Sheetfile" "POWER_MANAGEMENT.kicad_sch"
+			(at 107.95 164.4146 0)
+			(show_name no)
+			(do_not_autoplace no)
+			(effects
+				(font
+					(size 1.27 1.27)
+				)
+				(justify left top)
+			)
+		)
+		(instances
+			(project "robot_canettes"
+				(path "/67ea9330-6bd8-4bfd-bb5f-e77247705b59"
+					(page "3")
+				)
+			)
+		)
+	)
+	(sheet
+		(at 17.78 35.56)
+		(size 80.01 128.27)
+		(exclude_from_sim no)
+		(in_bom yes)
+		(on_board yes)
+		(dnp no)
+		(fields_autoplaced yes)
+		(stroke
+			(width 0.1524)
+			(type solid)
+		)
+		(fill
+			(color 0 0 0 0)
+		)
+		(property "Sheetname" "MCU_AND_SENSORS"
+			(at 17.78 34.8484 0)
+			(show_name no)
+			(do_not_autoplace no)
+			(effects
+				(font
+					(size 1.27 1.27)
+				)
+				(justify left bottom)
+			)
+		)
+		(property "Sheetfile" "MCU_AND_SENSORS.kicad_sch"
+			(at 17.78 164.4146 0)
+			(show_name no)
+			(do_not_autoplace no)
+			(effects
+				(font
+					(size 1.27 1.27)
+				)
+				(justify left top)
+			)
+		)
+		(instances
+			(project "robot_canettes"
+				(path "/67ea9330-6bd8-4bfd-bb5f-e77247705b59"
+					(page "2")
+				)
+			)
+		)
+	)
+	(sheet
+		(at 196.85 35.56)
+		(size 82.55 128.27)
+		(exclude_from_sim no)
+		(in_bom yes)
+		(on_board yes)
+		(dnp no)
+		(fields_autoplaced yes)
+		(stroke
+			(width 0.1524)
+			(type solid)
+		)
+		(fill
+			(color 0 0 0 0)
+		)
+		(property "Sheetname" "MOTOR_DRIVE"
+			(at 196.85 34.8484 0)
+			(show_name no)
+			(do_not_autoplace no)
+			(effects
+				(font
+					(size 1.27 1.27)
+				)
+				(justify left bottom)
+			)
+		)
+		(property "Sheetfile" "MOTOR_DRIVE.kicad_sch"
+			(at 196.85 164.4146 0)
+			(show_name no)
+			(do_not_autoplace no)
+			(effects
+				(font
+					(size 1.27 1.27)
+				)
+				(justify left top)
+			)
+		)
+		(instances
+			(project "robot_canettes"
+				(path "/67ea9330-6bd8-4bfd-bb5f-e77247705b59"
+					(page "4")
+				)
+			)
+		)
+	)
 	(sheet_instances
 		(path "/"

Commit message: MOTOR_DRIVE
Other:
- sheet MCU_AND_SENSORS renamed MCU
- added sheet SENSORS (SENSORS.kicad_sch)
- sheet MCU ports: added ESP32_RX, ESP32_TX, GAUGE_INT, I2C3_SCL, I2C3_SDA, INT, MOTOR_A_C1, MOTOR_A_C2, MOTOR_A_IN1, MOTOR_A_IN2, MOTOR_B_C1, MOTOR_B_C2, MOTOR_B_IN1, MOTOR_B_IN2, MOTOR_FAULT, MOTOR_SLEEP, MPU_INT, SERVO1_PWM; removed none
- sheet MOTOR_DRIVE ports: added MOTOR_A_C1, MOTOR_A_C2, MOTOR_A_IN1, MOTOR_A_IN2, MOTOR_B_C1, MOTOR_B_C2, MOTOR_B_IN1, MOTOR_B_IN2, MOTOR_FAULT, MOTOR_SLEEP, SERVO1_PWM, VM; removed none
- sheet POWER_MANAGEMENT ports: added GAUGE_INT, I2C3_SCL, I2C3_SDA, INT; removed none
