File: hardware/kicad/robot_canettes/robot_canettes.kicad_pcb (KiCad board)
At the start: 4 copper layers, 78 x 68 mm, 114 parts, among them J1 Conn_01x04_Pin, J10 Conn_01x06, J11 Conn_01x06, J12 Conn_01x06, J3 C573320, J4 USB_C_Receptacle_USB2.0_16P, J5 Conn_01x02_Pin, J6 Conn_01x03, J7 Conn_01x06, J8 Conn_01x06, J9 Conn_01x04_Pin, Q1 2N7002, Q2 Q_PMOS, Q5 Q_PNP_CurrentMirror, U1 STM32G431RBTx, U2 MPU-6050, U3 DRV8833PWP, U4 AP2112K-3.3, U5 bq27220, U6 SN74AHCT1G125DBVR, U9 BQ25896RTWR, Y1 16M

Commit message: Update robot PCB
Parts:
- moved J1 63.2 mm to (131.2, 127.0), turned to 180 degrees
- moved C43 58.6 mm to (132.2, 122.7), turned to 0 degrees
- moved C16 5.32 mm to (121.0, 116.0), turned to 180 degrees
- moved C17 3.31 mm to (127.8, 118.4), turned to 0 degrees
- moved R1 2.79 mm to (117.2, 108.0), turned to 180 degrees
- moved R21 2.44 mm to (86.7, 91.0), turned to -90 degrees
- moved Y1 2.38 mm to (124.4, 117.3), turned to -90 degrees
- moved C15 2.25 mm to (136.2, 107.0)
- moved C7 2.04 mm to (131.2, 114.2)
- moved C27 1.79 mm to (85.5, 91.9), turned to -90 degrees
- moved SW2 1.75 mm to (141.8, 111.0), turned to -90 degrees
- moved R15 1.47 mm to (95.8, 89.5)
- moved C42 1.41 mm to (110.0, 90.0)
- moved R6 1.21 mm to (90.8, 96.7)
- moved C32 1.03 mm to (99.0, 97.0), turned to 0 degrees
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Connections:
- J7 pad 2: GND -> <NO NET>
- U1 pad 13: /MCU/TOF1_XSHUT -> unconnected-(U1-PA1-Pad13)
- U1 pad 14: /MCU/TOF2_XSHUT -> unconnected-(U1-PA2-Pad14)
- U1 pad 34: unconnected-(U1-PB12-Pad34) -> /MCU/TOF1_XSHUT
- U1 pad 35: unconnected-(U1-PB13-Pad35) -> /MCU/TOF2_XSHUT
Routing:
- net /MCU/TOF2_INT: track 0.00 -> 94.3 mm, vias 0 -> 2
- net /MCU/INT: track 0.00 -> 70.3 mm, vias 0 -> 8
- net /MCU/TOF1_INT: track 0.00 -> 61.8 mm, vias 0 -> 4
- net /MCU/MOTOR_SLEEP: track 0.00 -> 56.5 mm, vias 0 -> 6
- net /MCU/MOTOR_FAULT: track 0.00 -> 53.4 mm, vias 0 -> 4
- net /MCU/MOTOR_B_C2: track 0.00 -> 52.5 mm, vias 0 -> 8
- net /MCU/MOTOR_B_C1: track 0.00 -> 52.5 mm, vias 0 -> 9
- net /MCU/TOF3_XSHUT: track 0.00 -> 48.8 mm, vias 0 -> 3
- net /MCU/I2C3_SDA: track 60.5 -> 108.6 mm, vias 6 -> 8
- net /MCU/TOF3_INT: track 0.00 -> 47.9 mm, vias 0 -> 4
- net VBUS: track 22.9 -> 70.5 mm
- net /MCU/TOF2_XSHUT: track 0.00 -> 46.2 mm, vias 0 -> 3
- net Net-(Q1-D): track 0.00 -> 46.0 mm, vias 0 -> 5
- net /MCU/ESP32_RX: track 70.6 -> 26.3 mm
- net /MCU/TOF1_XSHUT: track 0.00 -> 40.0 mm, vias 0 -> 3
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