File: hardware/kicad/robot_canettes/robot_canettes.kicad_pcb (KiCad board)
At the start: 4 copper layers, 78 x 68 mm, 114 parts, among them J1 Conn_01x04_Pin, J10 Conn_01x06, J11 Conn_01x06, J12 Conn_01x06, J3 C573320, J4 USB_C_Receptacle_USB2.0_16P, J5 Conn_01x02_Pin, J6 Conn_01x03, J7 Conn_01x06, J8 Conn_01x06, J9 Conn_01x04_Pin, Q1 2N7002, Q2 Q_PMOS, Q5 Q_PNP_CurrentMirror, U1 STM32G431RBTx, U2 MPU-6050, U3 DRV8833PWP, U4 AP2112K-3.3, U5 bq27220, U6 SN74AHCT1G125DBVR, U9 BQ25896RTWR, Y1 16M

Commit message: Mise à jour du PCB
Parts:
- moved C7 2.04 mm to (129.4, 113.4)
- moved C1 1.25 mm to (136.7, 103.5)
- moved C3 1.25 mm to (137.7, 103.5)
- moved C4 0.38 mm to (119.0, 99.6)
- moved H102 0.05 mm to (141.7, 66.1)
- renumbered J3 to APDS, J12 to TOF1, J10 to TOF2, J11 to TOF3
Connections:
- J7 pad 2: <NO NET> -> GND
- U1 pad 13: unconnected-(U1-PA1-Pad13) -> /MCU/TOF1_XSHUT
- U1 pad 14: unconnected-(U1-PA2-Pad14) -> /MCU/TOF2_XSHUT
- U1 pad 34: /MCU/TOF1_XSHUT -> unconnected-(U1-PB12-Pad34)
- U1 pad 35: /MCU/TOF2_XSHUT -> unconnected-(U1-PB13-Pad35)
Routing:
- net VBUS: track 70.5 -> 187.7 mm, vias 20 -> 9
- net /MCU/TOF2_INT: track 94.3 -> 4.26 mm, vias 2 -> 1
- net /MCU/TOF1_INT: track 61.8 -> 0.00 mm, vias 4 -> 0
- net /MCU/MOTOR_SLEEP: track 56.5 -> 110.6 mm, vias 6 -> 5
- net /MCU/TOF2_XSHUT: track 46.2 -> 3.25 mm, vias 3 -> 0
- net /MCU/TOF1_XSHUT: track 40.0 -> 0.00 mm, vias 3 -> 0
- net /MCU/GAUGE_INT: track 37.2 -> 3.61 mm, vias 3 -> 1
- net /MCU/ESP32_TX: track 32.1 -> 0.00 mm, vias 4 -> 0
- net /MCU/ESP32_RX: track 26.3 -> 0.00 mm, vias 2 -> 0
- net /MCU/I2C3_SCL: track 113.6 -> 90.2 mm
- net /MCU/I2C2_SDA: track 59.0 -> 35.9 mm, vias 2 -> 4
- net /MCU/I2C2_SCL: track 84.6 -> 106.0 mm, vias 2 -> 6
- net /MCU/INT: track 70.3 -> 52.6 mm, vias 8 -> 5
- net USB_5V: track 16.2 -> 31.6 mm, vias 2 -> 1
- net /MCU/SWDIO: track 31.4 -> 46.1 mm
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Other:
- outline, holes or cut-outs redrawn

Commit message: Mise à jour du PCB (routage)
Parts:
- moved R22 0.45 mm to (114.6, 78.8)
- moved C7 0.43 mm to (129.8, 113.5)
Routing:
- net /MCU/TOF1_XSHUT: track 0.00 -> 96.1 mm, vias 0 -> 4
- net /MCU/TOF2_XSHUT: track 3.25 -> 73.7 mm, vias 0 -> 2
- net /MCU/TOF1_INT: track 0.00 -> 54.4 mm
- net /MCU/I2C3_SCL: track 90.2 -> 70.4 mm
- net +3.3V: track 46.9 -> 55.6 mm, vias 41 -> 36
- net GND: track 108.0 -> 115.5 mm, vias 94 -> 90
- net /MCU/I2C3_SDA: track 111.6 -> 114.4 mm, vias 4 -> 5
- net /MCU/TOF2_INT: track 4.26 -> 2.05 mm
- net /MCU/I2C2_SCL: track 106.0 -> 104.4 mm

Commit message: Final PCB LAYOUT
Parts:
- moved C22 5.47 mm to (145.0, 81.0), turned to 90 degrees
- moved R27 2.87 mm to (81.5, 89.5), turned to -90 degrees
- moved TP_SDA_2 2.86 mm to (85.8, 96.6)
- moved C27 2.54 mm to (88.0, 91.2)
- moved C15 2.36 mm to (134.0, 106.2)
- moved TP_BAT1 1.89 mm to (73.6, 96.0)
- moved R21 1.66 mm to (87.5, 89.6), turned to 0 degrees
- moved C1 1.50 mm to (136.8, 105.0), turned to -90 degrees
- moved C3 1.50 mm to (137.8, 105.0), turned to -90 degrees
- moved TP_USB_5V1 1.32 mm to (78.9, 76.5)
- moved TP_SYS1 1.27 mm to (111.2, 79.8)
- moved C4 1.01 mm to (120.0, 99.8), turned to 180 degrees
- moved C40 1.00 mm to (126.0, 69.0)
- moved C5 1.00 mm to (117.8, 110.0)
- moved R5 0.90 mm to (79.0, 79.4)
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- renumbered J5 to Battery, J4 to Charging, J1 to ESP32, J7 to M1, J8 to M2, J9 to NEOPIXEL, J6 to Servo
Routing:
- net /MCU/TOF2_INT: track 2.05 -> 74.3 mm, vias 1 -> 4
- net VBUS: track 187.7 -> 134.9 mm, vias 9 -> 12
- net /MCU/ESP32_RX: track 0.00 -> 50.9 mm, vias 0 -> 4
- net /MCU/GAUGE_INT: track 3.61 -> 46.4 mm, vias 1 -> 4
- net /MCU/I2C3_SCL: track 70.4 -> 110.3 mm, vias 2 -> 8
- net /MCU/I2C2_SDA: track 35.9 -> 66.9 mm, vias 4 -> 6
- net /MCU/ESP32_TX: track 0.00 -> 29.2 mm
- net Net-(Q1-D): track 38.1 -> 60.2 mm, vias 3 -> 2
- net GND: track 115.5 -> 136.2 mm, vias 90 -> 81
- net +3.3V: track 55.6 -> 70.6 mm, vias 36 -> 28
- net /MCU/MOTOR_SLEEP: track 110.6 -> 122.9 mm, vias 5 -> 6
- net /MCU/I2C3_SDA: track 114.4 -> 104.0 mm, vias 5 -> 7
- net /MCU/TOF1_XSHUT: track 96.1 -> 89.1 mm
- net /MCU/TOF2_XSHUT: track 73.7 -> 68.2 mm
- net /MCU/TOF1_INT: track 54.4 -> 59.0 mm, vias 0 -> 2
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- added copper zone on F.Cu, net VBUS
Other:
- board text added: "+"
- board text added: "-"

Commit message: Mise a jour des schemas, layout final, routage et génération des fichiers de fabrication de la carte
Parts:
- moved G*** 3.28 mm to (123.9, 83.9)
- moved Battery1 2.65 mm to (70.7, 91.3), turned to 90 degrees
- moved C42 0.82 mm to (110.8, 90.2)
- moved R18 0.70 mm to (99.7, 122.0)
- moved R17 0.52 mm to (93.2, 122.1)
- moved Charging1 0.35 mm to (71.7, 80.0)
- renumbered APDS to APDS1, Battery to Battery1, Charging to Charging1, NEOPIXEL to NEOPIXEL1, Servo to Servo1
Routing:
- net USB_5V: track 28.0 -> 6.25 mm
- net Net-(J7-Pin_6): track 10.4 -> 0.00 mm
- net Net-(J7-Pin_1): track 10.2 -> 0.00 mm
- net Net-(J8-Pin_6): track 25.1 -> 19.2 mm
- net /MCU/MOTOR_SLEEP: track 122.9 -> 128.1 mm
- net +BATT: track 51.0 -> 54.9 mm
- net Net-(D1-K): track 21.7 -> 23.7 mm
- net /MCU/I2C3_SCL: track 110.3 -> 109.0 mm, vias 8 -> 7
- net Net-(Q1-D): track 60.2 -> 61.3 mm
- net Net-(J8-Pin_1): track 31.8 -> 30.8 mm
- net /MCU/TOF1_XSHUT: track 89.1 -> 90.1 mm
- net /MCU/TOF2_XSHUT: track 68.2 -> 69.0 mm
- net /MCU/I2C2_SDA: track 66.9 -> 67.7 mm
- net Net-(Q2-G): track 6.72 -> 7.52 mm
- net /POWER_MANAGEMENT/SRN: track 12.1 -> 12.8 mm
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- added copper zone on B.Cu, net GND
- added copper zone on F.Cu, net GND
- added copper zone on F.Cu, net Net-(J7-Pin_1)
- added copper zone on F.Cu, net Net-(J7-Pin_6)
- added copper zone on F.Cu, net Net-(J8-Pin_1)
- added copper zone on F.Cu, net Net-(J8-Pin_6)
- added copper zone on F.Cu, net USB_5V
