File: hardware/kicad/robot_canettes/SENSORS.kicad_sch (KiCad schematic)
At the start: 17 parts, among them J1 Conn_01x04_Pin, J10 Conn_01x06, J11 Conn_01x06, J2 Conn_01x06, J3 C573320, U2 MPU-6050

Commit message: Mise a jour du projet, correction du nom de la feuille sensors
Parts:
- removed J2: Conn_01x06, Connector_JST:JST_PH_B6B-PH-K_1x06_P2.00mm_Vertical, symbol Connector_Generic:Conn_01x06
- added J12: Conn_01x06, Connector_PinHeader_1.00mm:PinHeader_1x06_P1.00mm_Horizontal, symbol Connector_Generic:Conn_01x06
- J1: footprint Connector_JST:JST_PH_B4B-PH-K_1x04_P2.00mm_Vertical -> Connector_PinHeader_2.54mm:PinHeader_1x04_P2.54mm_Vertical
- J10, J11: footprint Connector_JST:JST_PH_B6B-PH-K_1x06_P2.00mm_Vertical -> Connector_PinHeader_1.00mm:PinHeader_1x06_P1.00mm_Horizontal
- J3: footprint Connector_JST:JST_PH_B5B-PH-K_1x05_P2.00mm_Vertical -> Connector_PinHeader_1.00mm:PinHeader_1x05_P1.00mm_Horizontal
Connections:
- net +3.3V: now also J12.1 (Pin_1)
- net I2C3_SCL: now also J12.3 (Pin_3)
- net I2C3_SDA: now also J12.4 (Pin_4)
- net TOF1_INT: now also J11.5 (Pin_5)
- net TOF1_XSHUT: now also J11.6 (Pin_6)
- net TOF3_INT: now also J12.5 (Pin_5); no longer J11.5 (Pin_5)
- net TOF3_XSHUT: now also J12.6 (Pin_6); no longer J11.6 (Pin_6)
- net at C40.2: now also J11.2 (Pin_2)
- net at C41.2: now also J12.2 (Pin_2); no longer J11.2 (Pin_2)

Commit message: Mise à jour de l'emplacement des composants
Parts:
- J1: footprint Connector_PinHeader_2.54mm:PinHeader_1x04_P2.54mm_Vertical -> Connector_JST:JST_PH_B4B-PH-K_1x04_P2.00mm_Vertical
- J10, J11, J12: footprint Connector_PinHeader_1.00mm:PinHeader_1x06_P1.00mm_Horizontal -> Connector_JST:JST_PH_B6B-PH-K_1x06_P2.00mm_Vertical
- J3: footprint Connector_PinHeader_1.00mm:PinHeader_1x05_P1.00mm_Horizontal -> Connector_JST:JST_PH_B5B-PH-K_1x05_P2.00mm_Vertical
Connections:
- net GND: now also C11.2, C12.2, C13.2, C14.2, C38.2, C39.2, C40.2, C41.2, J1.4 (Pin_4), J10.2 (Pin_2), J11.2 (Pin_2), J12.2 (Pin_2), J3.2 (Pin_2), U2.11 (FSYNC), U2.18 (GND), U2.9 (AD0)
Changed lines of the file:
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@@
 			)
 		)
-		(property "Value" ""
+		(property "Value" "GND"
 			(at 241.3 68.58 0)
+			(hide yes)
 			(show_name no)
 			(do_not_autoplace no)
@@
 			)
 		)
-		(property "Value" ""
+		(property "Value" "GND"
 			(at 140.97 67.31 0)
+			(hide yes)
 			(show_name no)
 			(do_not_autoplace no)
@@
 			)
 		)
-		(property "Value" ""
+		(property "Value" "GND"
 			(at 92.71 127 0)
+			(hide yes)
 			(show_name no)
 			(do_not_autoplace no)
@@
 			)
 		)
-		(property "Footprint" "Connector_PinHeader_2.54mm:PinHeader_1x04_P2.54mm_Vertical"
+		(property "Footprint" "Connector_JST:JST_PH_B4B-PH-K_1x04_P2.00mm_Vertical"
 			(at 193.04 137.16 0)
 			(hide yes)
@@
 			)
 		)
-		(property "Value" ""
+		(property "Value" "GND"
 			(at 38.1 107.95 0)
+			(hide yes)
 			(show_name no)
 			(do_not_autoplace no)
@@
 			)
 		)
-		(property "Footprint" "Connector_PinHeader_1.00mm:PinHeader_1x06_P1.00mm_Horizontal"
+		(property "Footprint" "Connector_JST:JST_PH_B6B-PH-K_1x06_P2.00mm_Vertical"
 			(at 161.29 62.23 0)
 			(hide yes)
@@
 			)
 		)
-		(property "Value" ""
+		(property "Value" "GND"
 			(at 201.93 147.32 0)
+			(hide yes)
 			(show_name no)
 			(do_not_autoplace no)
@@
 			)
 		)
-		(property "Value" ""
+		(property "Value" "GND"
 			(at 43.18 92.71 0)
+			(hide yes)
 			(show_name no)
 			(do_not_autoplace no)
@@
 			)
 		)
-		(property "Value" ""
+		(property "Value" "GND"
 			(at 85.09 127 0)
+			(hide yes)
 			(show_name no)
 			(do_not_autoplace no)
@@
 		(property "Value" "GND"
 			(at 210.82 139.7 0)
+			(hide yes)
 			(show_name no)
 			(do_not_autoplace no)
@@
 			)
 		)
-		(property "Footprint" "Connector_PinHeader_1.00mm:PinHeader_1x05_P1.00mm_Horizontal"
+		(property "Footprint" "Connector_JST:JST_PH_B5B-PH-K_1x05_P2.00mm_Vertical"
 			(at 265.43 64.77 0)
 			(hide yes)
@@
 			)
 		)
-		(property "Value" ""
+		(property "Value" "GND"
 			(at 62.23 128.27 0)
+			(hide yes)
 			(show_name no)
 			(do_not_autoplace no)
@@
 			)
 		)
-		(property "Footprint" "Connector_PinHeader_1.00mm:PinHeader_1x06_P1.00mm_Horizontal"
+		(property "Footprint" "Connector_JST:JST_PH_B6B-PH-K_1x06_P2.00mm_Vertical"
 			(at 158.75 134.62 0)
 			(hide yes)
@@
 			)
 		)
-		(property "Value" ""
+		(property "Value" "GND"
 			(at 77.47 91.44 0)
+			(hide yes)
 			(show_name no)
 			(do_not_autoplace no)
@@
 			)
 		)
-		(property "Footprint" "Connector_PinHeader_1.00mm:PinHeader_1x06_P1.00mm_Horizontal"
+		(property "Footprint" "Connector_JST:JST_PH_B6B-PH-K_1x06_P2.00mm_Vertical"
 			(at 213.36 62.23 0)
 			(hide yes)
@@
 			)
 		)
-		(property "Value" ""
+		(property "Value" "GND"
 			(at 193.04 67.31 0)
+			(hide yes)
 			(show_name no)
 			(do_not_autoplace no)
@@
 			)
 		)
-		(property "Value" ""
+		(property "Value" "GND"
 			(at 138.43 139.7 0)
-			(show_name no)
-			(do_not_autoplace no)
+			(hide yes)
+			(show_name no)
+			(do_not_autoplace no)

Commit message: Final PCB LAYOUT
Parts:
- J1: JLCPCB Part # (none) -> C131334
- J10, J11, J12: JLCPCB Part # (none) -> C131342
- J3: JLCPCB PART# C573320 -> C157993
Changed lines of the file:
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@@
+			)
+		)
+		(property "JLCPCB Part #" "C131334"
+			(at 193.04 137.16 0)
+			(hide yes)
+			(show_name no)
+			(do_not_autoplace no)
+			(effects
+				(font
+					(size 1.27 1.27)
+				)
 			)
 		)
@@
 		)
 		(property "Description" "Generic connector, single row, 01x06, script generated (kicad-library-utils/schlib/autogen/connector/)"
+			(at 161.29 62.23 0)
+			(hide yes)
+			(show_name no)
+			(do_not_autoplace no)
+			(effects
+				(font
+					(size 1.27 1.27)
+				)
+			)
+		)
+		(property "JLCPCB Part #" "C131342"
 			(at 161.29 62.23 0)
 			(hide yes)
@@
 			)
 		)
-		(property "JLCPCB PART#" "C573320"
+		(property "JLCPCB PART#" "C157993"
 			(at 265.43 64.77 0)
 			(hide yes)
@@
 		)
 		(property "Description" "Generic connector, single row, 01x06, script generated (kicad-library-utils/schlib/autogen/connector/)"
+			(at 158.75 134.62 0)
+			(hide yes)
+			(show_name no)
+			(do_not_autoplace no)
+			(effects
+				(font
+					(size 1.27 1.27)
+				)
+			)
+		)
+		(property "JLCPCB Part #" "C131342"
 			(at 158.75 134.62 0)
 			(hide yes)
@@
 			(at 213.36 62.23 0)
 			(hide yes)
+			(show_name no)
+			(do_not_autoplace no)
+			(effects
+				(font
+					(size 1.27 1.27)
+				)
+			)
+		)
+		(property "JLCPCB Part #" "C131342"
+			(at 213.36 62.23 0)
+			(hide yes)

Commit message: Mise a jour des schemas, layout final, routage et génération des fichiers de fabrication de la carte
Parts:
- APDS1: renamed from J3; value C573320 -> Conn_01x05; JLCPCB PART# C157993 -> (none); JLCPCB Part # (none) -> C157993
- C11: JLCPCB PART # C15195 -> (none); JLCPCB Part # (none) -> C15195
- C12: JLCPCB PART # C1531 -> (none); JLCPCB Part # (none) -> C1531
- C13, C14, C38, C39, C40, C41, C43: JLCPCB PART # C1525 -> (none); JLCPCB Part # (none) -> C1525
- R13, R2: JLCPCB PART # C174143 -> (none); JLCPCB Part # (none) -> C25879
- U2: JLCPCB PART # C24112 -> (none); JLCPCB Part # (none) -> C24112
- renumbered J1 to ESP32, J11 to TOF1, J10 to TOF2, J12 to TOF3
Changed lines of the file:
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@@
 		(dnp no)
 		(property "Reference" "C39"
-			(at 195.58 58.4199 0)
-			(hide yes)
+			(at 187.198 58.166 0)
 			(show_name no)
 			(do_not_autoplace no)
@@
 			)
 		)
-		(property "JLCPCB PART #" "C1525"
+		(property "JLCPCB Part #" "C1525"
 			(at 193.04 59.69 0)
 			(hide yes)
@@
 		(dnp no)
 		(fields_autoplaced yes)
-		(property "Reference" "J1"
+		(property "Reference" "ESP32"
 			(at 193.675 129.54 0)
 			(show_name no)
@@
 			(project "robot_canettes"
 				(path "/67ea9330-6bd8-4bfd-bb5f-e77247705b59/18019061-6b67-4462-b338-223d78003134"
-					(reference "J1")
+					(reference "ESP32")
 					(unit 1)
 				)
@@
 		(dnp no)
 		(fields_autoplaced yes)
-		(property "Reference" "J11"
+		(property "Reference" "TOF1"
 			(at 163.83 62.2299 0)
 			(show_name no)
@@
 			(project "robot_canettes"
 				(path "/67ea9330-6bd8-4bfd-bb5f-e77247705b59/18019061-6b67-4462-b338-223d78003134"
-					(reference "J11")
+					(reference "TOF1")
 					(unit 1)
 				)
@@
 			)
 		)
-		(property "JLCPCB PART #" "C1525"
+		(property "JLCPCB Part #" "C1525"
 			(at 85.09 119.38 0)
 			(hide yes)
@@
 			)
 		)
-		(property "JLCPCB PART #" "C174143"
+		(property "JLCPCB Part #" "C25879"
 			(at 267.97 130.81 0)
 			(hide yes)
@@
 			)
 		)
-		(property "JLCPCB PART #" "C1525"
+		(property "JLCPCB Part #" "C1525"
 			(at 241.3 59.69 0)
 			(hide yes)
@@
 		(dnp no)
 		(fields_autoplaced yes)
-		(property "Reference" "J3"
+		(property "Reference" "APDS1"
 			(at 267.97 63.4999 0)
 			(show_name no)
@@
 			)
 		)
-		(property "Value" "C573320"
+		(property "Value" "Conn_01x05"
 			(at 267.97 66.0399 0)
 			(show_name no)
@@
 			)
 		)
-		(property "JLCPCB PART#" "C157993"
+		(property "JLCPCB Part #" "C157993"
 			(at 265.43 64.77 0)
 			(hide yes)
@@
 			(project "robot_canettes"
 				(path "/67ea9330-6bd8-4bfd-bb5f-e77247705b59/18019061-6b67-4462-b338-223d78003134"
-					(reference "J3")
+					(reference "APDS1")
 					(unit 1)
 				)
@@
 			)
 		)
-		(property "JLCPCB PART #" "C1525"
+		(property "JLCPCB Part #" "C1525"
 			(at 77.47 83.82 0)
 			(hide yes)
@@
 		(dnp no)
 		(property "Reference" "C40"
-			(at 143.51 58.4199 0)
-			(hide yes)
+			(at 135.382 57.912 0)
 			(show_name no)
 			(do_not_autoplace no)
@@
 			)
 		)
-		(property "JLCPCB PART #" "C1525"
+		(property "JLCPCB Part #" "C1525"
 			(at 140.97 59.69 0)
 			(hide yes)
@@
 		(dnp no)
 		(fields_autoplaced yes)
-		(property "Reference" "J12"
+		(property "Reference" "TOF3"
 			(at 161.29 134.6199 0)
 			(show_name no)
@@
 			(project "robot_canettes"
 				(path "/67ea9330-6bd8-4bfd-bb5f-e77247705b59/18019061-6b67-4462-b338-223d78003134"
-					(reference "J12")
+					(reference "TOF3")
 					(unit 1)
 				)
@@
 		(property "Reference" "C43"
 			(at 213.36 130.8099 0)
-			(hide yes)
 			(show_name no)
 			(do_not_autoplace no)
@@
 			)
 		)
-		(property "JLCPCB PART #" "C1525"
+		(property "JLCPCB Part #" "C1525"
 			(at 210.82 132.08 0)
 			(hide yes)
@@
 		(dnp no)
 		(property "Reference" "C41"
-			(at 140.97 130.8099 0)
-			(hide yes)
+			(at 133.096 130.302 0)
 			(show_name no)
 			(do_not_autoplace no)
@@
 			)
 		)
-		(property "JLCPCB PART #" "C1525"
+		(property "JLCPCB Part #" "C1525"
 			(at 138.43 132.08 0)
 			(hide yes)
@@
 			)
 		)
-		(property "JLCPCB PART #" "C24112"
+		(property "JLCPCB Part #" "C24112"
 			(at 62.23 105.41 0)
 			(hide yes)
@@
 			)
 		)
-		(property "JLCPCB PART #" "C174143"
+		(property "JLCPCB Part #" "C25879"
 			(at 260.35 130.81 0)
 			(hide yes)
@@
 		(dnp no)
 		(fields_autoplaced yes)
-		(property "Reference" "J10"
+		(property "Reference" "TOF2"
 			(at 215.9 62.2299 0)
 			(show_name no)
@@
 			(project "robot_canettes"
 				(path "/67ea9330-6bd8-4bfd-bb5f-e77247705b59/18019061-6b67-4462-b338-223d78003134"
-					(reference "J10")
+					(reference "TOF2")
 					(unit 1)
 				)
@@
 			)
 		)
-		(property "JLCPCB PART #" "C15195"
+		(property "JLCPCB Part #" "C15195"
 			(at 43.18 85.09 0)
 			(hide yes)
@@
 			)
 		)
-		(property "JLCPCB PART #" "C1531"
+		(property "JLCPCB Part #" "C1531"
 			(at 92.71 119.38 0)
 			(hide yes)
